File: ScannerBoard-Revised/satscanner.sch (KiCad schematic (older format))
At the start: 30 parts, among them CON1 LNB Power 22V, P1 F_Connector, U1 LNBP12SP, U2 MAX2015, U3 LT1019, U4 LTC2440, U5 L4931, U6 LTC2050

Commit message: Correct value for R2
Parts:
- R2: value 53 -> 43
Changed lines of the file:
@@
 P 7600 3850
 F 0 "R2" V 7392 3850 50  0000 C CNN
-F 1 "53" V 7483 3850 50  0000 C CNN
+F 1 "43" V 7483 3850 50  0000 C CNN
 F 2 "Resistors_SMD:R_0805" H 7600 3850 60  0001 C CNN
 F 3 "" H 7600 3850 60  0000 C CNN
